File: examples/Example_Heart.kicad_pcb (KiCad board)
At the start: 2 copper layers, 48.6 x 48.5 mm, 27 parts, among them SW1 BTN, SW2 BTN, U1 ATtiny85

Commit message: Корпуса деталей на 2D-виде платы, надпись by_Madamin, LICENSE.md
- вкладка «Плата»: детали рисуются сверху теми же моделями, что на «3D»
  (Показывать / Полупрозрачные / Скрыть в панели справа)
- плата EasyEDA: слой 3DModel включён — контуры корпусов видны в 2D
- by_Madamin на шелкографии всех плат-примеров
- LICENSE.md (MIT)

Co-Authored-By: Claude Opus 5.5 <noreply@anthropic.com>
Other:
- board text added: "by_Madamin"
Changed lines of the file:
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@@
   (gr_text "+5V" (at 36.8 7 0) (layer "F.SilkS") (effects (font (size 1 1) (thickness 0.15))))
   (gr_text "Heart V1.1" (at 43.8 20 90) (layer "B.SilkS") (effects (font (size 1.2 1.2) (thickness 0.15)) (justify mirror)))
+  (gr_text "by_Madamin" (at 7.2 20.6 90) (layer "F.SilkS") (effects (font (size 1 1) (thickness 0.15))))
 )
